File: hardware/gameflopMB_1/gameflopMB_1.kicad_sch (KiCad schematic)
At the start: 0 parts

Commit message: new push
Other:
- sheet Driver renamed Driver0
- sheet Alim ports: added GND; removed none
- sheet Driver0 ports: added GND; removed none
- sheet Driver1 ports: added GND; removed none
- sheet Driver2 ports: added GND; removed none
- sheet Driver3 ports: added GND; removed none
- sheet STM32 Page ports: added GND; removed none
Changed lines of the file:
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@@
 	(paper "A4")
 	(junction
+		(at 226.06 152.4)
+		(diameter 0)
+		(color 0 0 0 0)
+	)
+	(junction
 		(at 177.8 85.09)
 		(diameter 0)
@@
 	)
 	(junction
+		(at 120.65 124.46)
+		(diameter 0)
+		(color 0 0 0 0)
+	)
+	(junction
 		(at 185.42 81.28)
 		(diameter 0)
@@
 	)
 	(junction
+		(at 120.65 152.4)
+		(diameter 0)
+		(color 0 0 0 0)
+	)
+	(junction
 		(at 185.42 40.64)
 		(diameter 0)
@@
 	)
 	(junction
+		(at 172.72 152.4)
+		(diameter 0)
+		(color 0 0 0 0)
+	)
+	(junction
 		(at 186.69 85.09)
 		(diameter 0)
@@
 	(wire
 		(pts
+			(xy 172.72 152.4) (xy 226.06 152.4)
+		)
+		(stroke
+			(width 0)
+			(type default)
+		)
+	)
+	(wire
+		(pts
 			(xy 223.52 114.3) (xy 223.52 140.97)
 		)
@@
 	(wire
 		(pts
+			(xy 120.65 152.4) (xy 120.65 124.46)
+		)
+		(stroke
+			(width 0)
+			(type default)
+		)
+	)
+	(wire
+		(pts
+			(xy 278.13 62.23) (xy 278.13 152.4)
+		)
+		(stroke
+			(width 0)
+			(type default)
+		)
+	)
+	(wire
+		(pts
 			(xy 223.52 140.97) (xy 170.18 140.97)
 		)
@@
 	(wire
 		(pts
+			(xy 226.06 125.73) (xy 226.06 152.4)
+		)
+		(stroke
+			(width 0)
+			(type default)
+		)
+	)
+	(wire
+		(pts
+			(xy 173.99 124.46) (xy 172.72 124.46)
+		)
+		(stroke
+			(width 0)
+			(type default)
+		)
+	)
+	(wire
+		(pts
 			(xy 238.76 85.09) (xy 186.69 85.09)
 		)
@@
 	(wire
 		(pts
+			(xy 278.13 152.4) (xy 226.06 152.4)
+		)
+		(stroke
+			(width 0)
+			(type default)
+		)
+	)
+	(wire
+		(pts
+			(xy 91.44 152.4) (xy 120.65 152.4)
+		)
+		(stroke
+			(width 0)
+			(type default)
+		)
+	)
+	(wire
+		(pts
 			(xy 185.42 40.64) (xy 198.12 40.64)
 		)
@@
 	(wire
 		(pts
+			(xy 120.65 52.07) (xy 120.65 124.46)
+		)
+		(stroke
+			(width 0)
+			(type default)
+		)
+	)
+	(wire
+		(pts
 			(xy 153.67 85.09) (xy 153.67 91.44)
 		)
@@
 	(wire
 		(pts
+			(xy 120.65 124.46) (xy 124.46 124.46)
+		)
+		(stroke
+			(width 0)
+			(type default)
+		)
+	)
+	(wire
+		(pts
 			(xy 173.99 115.57) (xy 170.18 115.57)
 		)
@@
 	(wire
 		(pts
+			(xy 233.68 62.23) (xy 278.13 62.23)
+		)
+		(stroke
+			(width 0)
+			(type default)
+		)
+	)
+	(wire
+		(pts
+			(xy 125.73 52.07) (xy 120.65 52.07)
+		)
+		(stroke
+			(width 0)
+			(type default)
+		)
+	)
+	(wire
+		(pts
+			(xy 227.33 125.73) (xy 226.06 125.73)
+		)
+		(stroke
+			(width 0)
+			(type default)
+		)
+	)
+	(wire
+		(pts
 			(xy 110.49 140.97) (xy 110.49 115.57)
 		)
@@
 	(wire
 		(pts
+			(xy 172.72 124.46) (xy 172.72 152.4)
+		)
+		(stroke
+			(width 0)
+			(type default)
+		)
+	)
+	(wire
+		(pts
 			(xy 185.42 40.64) (xy 185.42 81.28)
 		)
@@
 		(pts
 			(xy 186.69 91.44) (xy 186.69 85.09)
+		)
+		(stroke
+			(width 0)
+			(type default)
+		)
+	)
+	(wire
+		(pts
+			(xy 120.65 152.4) (xy 172.72 152.4)
 		)
 		(stroke
@@
 			)
 		)
+		(pin "GND" input
+			(at 227.33 125.73 180)
+			(effects
+				(font
+					(size 1.27 1.27)
+				)
+				(justify left)
+			)
+		)
 		(instances
 			(project "gameflopMB_1"
@@
 			)
 		)
+		(pin "GND" input
+			(at 173.99 124.46 180)
+			(effects
+				(font
+					(size 1.27 1.27)
+				)
+				(justify left)
+			)
+		)
 		(instances
 			(project "gameflopMB_1"
@@
 			(color 0 0 0 0.0000)
 		)
-		(property "Sheetname" "Driver"
+		(property "Sheetname" "Driver0"
 			(at 125.73 27.2284 0)
 			(effects
@@
 		(pin "+5V" input
 			(at 125.73 43.18 180)
+			(effects
+				(font
+					(size 1.27 1.27)
+				)
+				(justify left)
+			)
+		)
+		(pin "GND" input
+			(at 125.73 52.07 180)
 			(effects
 				(font
@@
 			)
 		)
+		(pin "GND" input
+			(at 91.44 152.4 0)
+			(effects
+				(font
+					(size 1.27 1.27)
+				)
+				(justify right)
+			)
+		)
 		(instances
 			(project "gameflopMB_1"
@@
 			)
 		)
+		(pin "GND" input
+			(at 124.46 124.46 180)
+			(effects
+				(font
+					(size 1.27 1.27)
+				)
+				(justify left)
+			)
+		)
 		(instances
 			(project "gameflopMB_1"
@@
 			)
 		)
+		(pin "GND" input
+			(at 233.68 62.23 0)
+			(effects
+				(font
+					(size 1.27 1.27)
+				)
+				(justify right)
+			)
+		)

Commit message: new push
Other:
- sheet Audio ports: added 3,3V, GND; removed none
- note removed: "Driver LED"
Changed lines of the file:
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@@
+	)
+	(junction
+		(at 97.79 152.4)
+		(diameter 0)
+		(color 0 0 0 0)
 	)
 	(junction
@@
 		(color 0 0 0 0)
 	)
+	(junction
+		(at 100.33 81.28)
+		(diameter 0)
+		(color 0 0 0 0)
+	)
 	(wire
 		(pts
@@
 	(wire
 		(pts
+			(xy 19.05 181.61) (xy 97.79 181.61)
+		)
+		(stroke
+			(width 0)
+			(type default)
+		)
+	)
+	(wire
+		(pts
+			(xy 19.05 80.01) (xy 19.05 181.61)
+		)
+		(stroke
+			(width 0)
+			(type default)
+		)
+	)
+	(wire
+		(pts
 			(xy 278.13 62.23) (xy 278.13 152.4)
 		)
@@
 	(wire
 		(pts
+			(xy 97.79 152.4) (xy 120.65 152.4)
+		)
+		(stroke
+			(width 0)
+			(type default)
+		)
+	)
+	(wire
+		(pts
 			(xy 170.18 115.57) (xy 170.18 140.97)
 		)
@@
 	(wire
 		(pts
-			(xy 91.44 152.4) (xy 120.65 152.4)
+			(xy 91.44 152.4) (xy 97.79 152.4)
 		)
 		(stroke
@@
 	(wire
 		(pts
+			(xy 78.74 81.28) (xy 100.33 81.28)
+		)
+		(stroke
+			(width 0)
+			(type default)
+		)
+	)
+	(wire
+		(pts
 			(xy 170.18 140.97) (xy 110.49 140.97)
 		)
@@
 	(wire
 		(pts
+			(xy 25.4 80.01) (xy 19.05 80.01)
+		)
+		(stroke
+			(width 0)
+			(type default)
+		)
+	)
+	(wire
+		(pts
 			(xy 110.49 140.97) (xy 110.49 115.57)
 		)
@@
 	(wire
 		(pts
+			(xy 100.33 81.28) (xy 100.33 21.59)
+		)
+		(stroke
+			(width 0)
+			(type default)
+		)
+	)
+	(wire
+		(pts
 			(xy 177.8 38.1) (xy 177.8 85.09)
 		)
@@
 	(wire
 		(pts
-			(xy 100.33 127) (xy 100.33 21.59)
+			(xy 100.33 127) (xy 100.33 81.28)
 		)
 		(stroke
@@
 	(wire
 		(pts
+			(xy 97.79 181.61) (xy 97.79 152.4)
+		)
+		(stroke
+			(width 0)
+			(type default)
+		)
+	)
+	(wire
+		(pts
 			(xy 238.76 92.71) (xy 238.76 85.09)
 		)
@@
 			(width 0)
 			(type default)
-		)
-	)
-	(text "Driver LED"
-		(exclude_from_sim no)
-		(at 180.34 25.4 0)
-		(effects
-			(font
-				(size 1.27 1.27)
-			)
 		)
 	)
@@
 			)
 		)
+		(pin "3,3V" input
+			(at 78.74 81.28 0)
+			(effects
+				(font
+					(size 1.27 1.27)
+				)
+				(justify right)
+			)
+		)
+		(pin "GND" input
+			(at 25.4 80.01 180)
+			(effects
+				(font
+					(size 1.27 1.27)
+				)
+				(justify left)
+			)
+		)

Commit message: new push
Other:
- sheet Audio ports: added I2C_SCL, I2C_SDA; removed none
- sheet STM32 Page ports: added Codec_SCL, Codec_SDA; removed none
Changed lines of the file:
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@@
+	(wire
+		(pts
+			(xy 237.49 17.78) (xy 237.49 39.37)
+		)
+		(stroke
+			(width 0)
+			(type default)
+		)
+	)
 	(wire
 		(pts
@@
 	(wire
 		(pts
+			(xy 83.82 53.34) (xy 83.82 15.24)
+		)
+		(stroke
+			(width 0)
+			(type default)
+		)
+	)
+	(wire
+		(pts
 			(xy 120.65 152.4) (xy 120.65 124.46)
 		)
@@
 	(wire
 		(pts
+			(xy 83.82 15.24) (xy 242.57 15.24)
+		)
+		(stroke
+			(width 0)
+			(type default)
+		)
+	)
+	(wire
+		(pts
 			(xy 19.05 181.61) (xy 97.79 181.61)
 		)
@@
 	(wire
 		(pts
+			(xy 237.49 39.37) (xy 233.68 39.37)
+		)
+		(stroke
+			(width 0)
+			(type default)
+		)
+	)
+	(wire
+		(pts
 			(xy 97.79 152.4) (xy 120.65 152.4)
 		)
@@
 	(wire
 		(pts
+			(xy 78.74 53.34) (xy 83.82 53.34)
+		)
+		(stroke
+			(width 0)
+			(type default)
+		)
+	)
+	(wire
+		(pts
 			(xy 91.44 152.4) (xy 97.79 152.4)
 		)
@@
 	(wire
 		(pts
+			(xy 92.71 17.78) (xy 237.49 17.78)
+		)
+		(stroke
+			(width 0)
+			(type default)
+		)
+	)
+	(wire
+		(pts
 			(xy 177.8 85.09) (xy 153.67 85.09)
 		)
@@
 	(wire
 		(pts
+			(xy 233.68 43.18) (xy 242.57 43.18)
+		)
+		(stroke
+			(width 0)
+			(type default)
+		)
+	)
+	(wire
+		(pts
 			(xy 120.65 124.46) (xy 124.46 124.46)
 		)
@@
 	(wire
 		(pts
+			(xy 242.57 15.24) (xy 242.57 43.18)
+		)
+		(stroke
+			(width 0)
+			(type default)
+		)
+	)
+	(wire
+		(pts
 			(xy 227.33 125.73) (xy 226.06 125.73)
 		)
@@
 	(wire
 		(pts
+			(xy 78.74 57.15) (xy 92.71 57.15)
+		)
+		(stroke
+			(width 0)
+			(type default)
+		)
+	)
+	(wire
+		(pts
 			(xy 110.49 140.97) (xy 110.49 115.57)
 		)
@@
 		(pts
 			(xy 158.75 91.44) (xy 158.75 81.28)
+		)
+		(stroke
+			(width 0)
+			(type default)
+		)
+	)
+	(wire
+		(pts
+			(xy 92.71 57.15) (xy 92.71 17.78)
 		)
 		(stroke
@@
 			)
 		)
+		(pin "I2C_SDA" input
+			(at 78.74 57.15 0)
+			(effects
+				(font
+					(size 1.27 1.27)
+				)
+				(justify right)
+			)
+		)
+		(pin "I2C_SCL" input
+			(at 78.74 53.34 0)
+			(effects
+				(font
+					(size 1.27 1.27)
+				)
+				(justify right)
+			)
+		)
 		(instances
 			(project "gameflopMB_1"
@@
 			(effects
 				(font
+					(size 1.27 1.27)
+				)
+				(justify right)
+			)
+		)
+		(pin "Codec_SDA" input
+			(at 233.68 39.37 0)
+			(effects
+				(font
+					(size 1.27 1.27)
+				)
+				(justify right)
+			)
+		)
+		(pin "Codec_SCL" input
+			(at 233.68 43.18 0)
+			(effects
+				(font
