File: hardware/gameflopMB_1/Driver.kicad_sch (KiCad schematic)
At the start: 5 parts, among them IC1 HTK16K33

Commit message: new push
Parts:
- R5, R9: value 2.2k -> 4,7k
Connections:
- net +3.3V is gone; now on net +5V: R5.1, R9.1

Commit message: new push
Parts:
- removed IC1: HTK16K33, HT16K33:HT16K33, symbol HT16K33:HT16K33
- added IC2: HTK16K33, Library:HT16K33, symbol HT16K33:HT16K33
- C3: footprint (none) -> Capacitor_SMD:C_0805_2012Metric_Pad1.18x1.45mm_HandSolder
- R5, R9: footprint (none) -> Resistor_SMD:R_0805_2012Metric_Pad1.20x1.40mm_HandSolder
- U3: footprint (none) -> Library:BL-M12X883
Connections:
- net +5V: now also IC2.24 (VDD)
- net GND: now also IC2.1 (VSS)
- net SCL: now also IC2.22 (ROW0/A2)
- net SDA: now also IC2.23 (SDA)
- net at U3.1 (Pin1): now also IC2.7 (ROW15/K13)
- net at U3.10 (Pin10): now also IC2.13 (ROW9/K7)
- net at U3.11 (Pin11): now also IC2.14 (ROW8/K6)
- net at U3.12 (Pin12): now also IC2.2 (COM0/AD)
- net at U3.13 (Pin13): now also IC2.6 (COM7)
- net at U3.14 (Pin14): now also IC2.15 (ROW7/K5)
- net at U3.15 (Pin15): now also IC2.16 (ROW6/K4)
- net at U3.16 (Pin16): now also IC2.27 (COM6)
- net at U3.17 (Pin17): now also IC2.17 (ROW5/K3)
- net at U3.18 (Pin18): now also IC2.18 (ROW4/K2)
- net at U3.19 (Pin19): now also IC2.26 (COM5)
- net at U3.2 (Pin2): now also IC2.8 (ROW14/K12)
- net at U3.20 (Pin20): now also IC2.19 (ROW3/K1)
- net at U3.21 (Pin21): now also IC2.20 (ROW2/A0)
- net at U3.22 (Pin22): now also IC2.25 (COM4)
- net at U3.23 (Pin23): now also IC2.21 (ROW1/A1)
- net at U3.24 (Pin24): now also IC2.22 (ROW0/A2)
- net at U3.3 (Pin3): now also IC2.5 (COM3/KS2)
- net at U3.4 (Pin4): now also IC2.9 (ROW13/K11)
- net at U3.5 (Pin5): now also IC2.10 (ROW12/K10)
- net at U3.6 (Pin6): now also IC2.4 (COM2/KS1)
- net at U3.7 (Pin7): now also IC2.11 (ROW11/K9)
- net at U3.8 (Pin8): now also IC2.12 (ROW10/K8)
- net at U3.9 (Pin9): now also IC2.3 (COM1/KS0)
Changed lines of the file:
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@@
 			)
 		)
-		(property "Footprint" ""
+		(property "Footprint" "Library:BL-M12X883"
 			(at 191.77 111.76 0)
 			(effects
@@
 			)
 		)
-		(property "Footprint" ""
+		(property "Footprint" "Resistor_SMD:R_0805_2012Metric_Pad1.20x1.40mm_HandSolder"
 			(at 62.992 68.58 90)
 			(effects
@@
 			)
 		)
-		(property "Footprint" ""
+		(property "Footprint" "Capacitor_SMD:C_0805_2012Metric_Pad1.18x1.45mm_HandSolder"
 			(at 32.7152 39.37 0)
 			(effects
@@
 			)
 		)
-		(property "Footprint" ""
+		(property "Footprint" "Resistor_SMD:R_0805_2012Metric_Pad1.20x1.40mm_HandSolder"
 			(at 69.342 73.66 90)
 			(effects
@@
 	)
 	(symbol
+		(lib_name "HT16K33_1")
 		(lib_id "HT16K33:HT16K33")
 		(at 106.68 91.44 0)
@@
 		(on_board yes)
 		(dnp no)
-		(property "Reference" "IC1"
-			(at 106.426 59.436 0)
+		(fields_autoplaced yes)
+		(property "Reference" "IC2"
+			(at 106.68 58.42 0)
 			(effects
 				(font
@@
 		)
 		(property "Value" "HTK16K33"
-			(at 106.934 63.246 0)
-			(effects
-				(font
-					(size 1.27 1.27)
-				)
-				(justify bottom)
-			)
-		)
-		(property "Footprint" "HT16K33:HT16K33"
+			(at 106.68 60.96 0)
+			(effects
+				(font
+					(size 1.27 1.27)
+				)
+			)
+		)
+		(property "Footprint" "Library:HT16K33"
 			(at 106.68 91.44 0)
 			(effects
@@
 			)
 		)
+		(pin "26"
+		)
+		(pin "16"
+		)
+		(pin "5"
+		)
+		(pin "15"
+		)
+		(pin "22"
+		)
+		(pin "12"
+		)
+		(pin "25"
+		)
+		(pin "22"
+		)
+		(pin "13"
+		)
+		(pin "18"
+		)
+		(pin "24"
+		)
+		(pin "2"
+		)
+		(pin "1"
+		)
+		(pin "19"
+		)
 		(pin "17"
 		)
-		(pin "22"
+		(pin "8"
+		)
+		(pin "9"
+		)
+		(pin "27"
+		)
+		(pin "10"
+		)
+		(pin "14"
+		)
+		(pin "6"
+		)
+		(pin "4"
 		)
 		(pin "7"
 		)
-		(pin "6"
-		)
-		(pin "10"
-		)
-		(pin "14"
-		)
-		(pin "13"
+		(pin "11"
 		)
 		(pin "21"
 		)
-		(pin "12"
-		)
-		(pin "19"
-		)
-		(pin "8"
-		)
-		(pin "22"
+		(pin "20"
+		)
+		(pin "23"
 		)
 		(pin "3"
-		)
-		(pin "24"
-		)
-		(pin "2"
-		)
-		(pin "23"
-		)
-		(pin "1"
-		)
-		(pin "20"
-		)
-		(pin "11"
-		)
-		(pin "5"
-		)
-		(pin "8"
-		)
-		(pin "18"
-		)
-		(pin "15"
-		)
-		(pin "9"
-		)
-		(pin "9"
-		)
-		(pin "16"
-		)
-		(pin "4"
-		)
-		(pin "7"
 		)
 		(instances
 			(project "gameflopMB_1"
 				(path "/1784a7ba-5cb6-4933-8b46-757da711e3a0/585eda5f-c3be-48fc-88f5-d02597212ccf"
-					(reference "IC1")
+					(reference "IC2")
 					(unit 1)
 				)
 				(path "/1784a7ba-5cb6-4933-8b46-757da711e3a0/c59feacd-8f83-49a0-84e1-4d8cf4d90032"
-					(reference "IC3")
+					(reference "IC6")
 					(unit 1)
 				)
 				(path "/1784a7ba-5cb6-4933-8b46-757da711e3a0/3b812121-84e0-4fb6-b484-e478d0056e2a"
-					(reference "IC4")
+					(reference "IC7")
 					(unit 1)
 				)
 				(path "/1784a7ba-5cb6-4933-8b46-757da711e3a0/370b33f5-0f9b-48b8-8313-c2e66ae7233b"
-					(reference "IC5")
-					(unit 1)
-				)
+					(reference "IC8")
+					(unit 1)
+				)

Commit message: commit
Parts:
- C3: footprint Capacitor_SMD:C_0805_2012Metric_Pad1.18x1.45mm_HandSolder -> Capacitor_SMD:C_0603_1608Metric_Pad1.08x0.95mm_HandSolder
Changed lines of the file:
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@@
 			)
 		)
-		(property "Footprint" "Capacitor_SMD:C_0805_2012Metric_Pad1.18x1.45mm_HandSolder"
+		(property "Footprint" "Capacitor_SMD:C_0603_1608Metric_Pad1.08x0.95mm_HandSolder"
 			(at 32.7152 39.37 0)
 			(effects
