File: hardware/gameflopMB_1/STM32.kicad_sch (KiCad schematic)
At the start: 8 parts, among them J3 Micro_SD_Card, U11 STM32G431RBT6

Commit message: new push
Parts:
- added ButtonA, ButtonB, DOWN, LEFT, RIGHT, Select, Start, UP: ~, symbol New_Library:Switch carré
- added J5: Conn_02x07_Odd_Even, symbol Connector_Generic:Conn_02x07_Odd_Even
- added R15: 1k, symbol Device:R
Connections:
- net GND: now also J5.11 (Pin_11), J5.5 (Pin_5), J5.7 (Pin_7), R15.2
- net NRST: now also J5.12 (Pin_12)
- net USART2_TX: now reaches U11.14 (PA2)
- net USART2_TX: now also J5.14 (Pin_14)
- net USART2_RX: now reaches U11.17 (PA3)
- net USART2_RX: now also J5.13 (Pin_13)
- net SWDIO: now reaches U11.49 (PA13)
- net SWDIO: now also J5.4 (Pin_4)
- net SWDCK: now reaches U11.50 (PA14)
- net SWDCK: now also J5.6 (Pin_6)
- new net: DOWN.1 (Vin), DOWN.3 (Vout1)
- new net: RIGHT.1 (Vin), RIGHT.3 (Vout1)
- new net: UP.1 (Vin), UP.3 (Vout1)
- new net: ButtonA.1 (Vin), ButtonA.3 (Vout1)
- new net: LEFT.1 (Vin), LEFT.3 (Vout1)
- new net: ButtonB.1 (Vin), ButtonB.3 (Vout1)
- new net +3.3V: J5.3 (Pin_3), Select.1 (Vin), Select.3 (Vout1), Start.1 (Vin), Start.3 (Vout1)
- new net Select: R15.1, Select.2 (Vout2), Start.2 (Vout2)
- no-connect marks 0 -> 5

Commit message: new push
Parts:
- removed ButtonA, ButtonB, DOWN, LEFT, RIGHT, Select, Start, UP: ~, symbol New_Library:Switch carré
- added R16, R17: 4,7k, symbol Device:R
- added U12, U13, U14, U15, U16, U17, U18, U19: ~, symbol New_Library:Switch carré
- R15: value 1k -> 4,7k
Connections:
- net Select is gone; now on net +3.3V: R15.1
- net +3,3V: now also U12.3 (VIn3), U13.3 (VIn3), U14.3 (VIn3), U15.3 (VIn3), U16.3 (VIn3), U17.3 (VIn3), U18.3 (VIn3), U19.3 (VIn3)
- net +3.3V: now also J3.4 (VDD), R16.1, R17.1
- net GND: now also J3.6 (VSS), J3.9 (SHIELD); no longer R15.2
- net SPI1_SCK: now reaches U11.19 (PA5)
- net SPI1_SCK: now also J3.5 (CLK), R16.2
- net SPI1_MISO: now reaches U11.20 (PA6)
- net SPI1_MISO: now also J3.7 (DAT0), R15.2
- net SPI1_MOSI: now reaches U11.21 (PA7)
- net SPI1_MOSI: now also J3.3 (CMD), R17.2
- net SelectO: now reaches U11.30 (PB10)
- net SelectO: now also U18.2 (VOut)
- net StartO: now reaches U11.33 (PB11)
- net StartO: now also U19.2 (VOut)
- net A: now reaches U11.56 (PB3)
- net A: now also U12.2 (VOut)
- net B: now reaches U11.57 (PB4)
- net B: now also U13.2 (VOut)
- net Up: now reaches U11.58 (PB5)
- net Up: now also U14.2 (VOut)
- net Left: now reaches U11.59 (PB6)
- net Left: now also U15.2 (VOut)
- net Down: now reaches U11.60 (PB7)
- net Down: now also U16.2 (VOut)
- net Right: now reaches U11.62 (PB9)
- net Right: now also U17.2 (VOut)
- no-connect marks 5 -> 51
Other:
- moved on the sheet: C1, J3, J5

Commit message: new push
Parts:
- C1: value C_Small -> 100nF; footprint (none) -> Capacitor_SMD:C_0805_2012Metric_Pad1.18x1.45mm_HandSolder
- C12, C13, C14, C15, C2: footprint (none) -> Capacitor_SMD:C_0805_2012Metric_Pad1.18x1.45mm_HandSolder
- J3: footprint (none) -> Connector_Card:microSD_HC_Molex_104031-0811
- J5: footprint (none) -> Connector_PinHeader_1.27mm:PinHeader_2x07_P1.27mm_Vertical
- R15, R16, R17: footprint (none) -> Resistor_SMD:R_0805_2012Metric_Pad1.20x1.40mm_HandSolder
- U12, U13, U14, U15, U16, U17, U18, U19: footprint (none) -> Library:Switch carré
Connections:
- net Codec_SCL: now reaches U11.22 (PC4)
- net Codec_SDA: now reaches U11.5 (PF0)
- no-connect marks 51 -> 49
Changed lines of the file:
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@@
 	)
 	(no_connect
-		(at 130.81 86.36)
-	)
-	(no_connect
 		(at 234.95 68.58)
 	)
@@
 	)
 	(no_connect
+		(at 130.81 93.98)
+	)
+	(no_connect
 		(at 166.37 127)
 	)
@@
 	)
 	(no_connect
-		(at 130.81 93.98)
-	)
-	(no_connect
-		(at 130.81 63.5)
-	)
-	(no_connect
 		(at 57.15 83.82)
 	)
@@
 	(wire
 		(pts
+			(xy 120.65 86.36) (xy 130.81 86.36)
+		)
+		(stroke
+			(width 0)
+			(type default)
+		)
+	)
+	(wire
+		(pts
 			(xy 210.82 119.38) (xy 210.82 121.92)
 		)
@@
 	(wire
 		(pts
+			(xy 121.92 63.5) (xy 130.81 63.5)
+		)
+		(stroke
+			(width 0)
+			(type default)
+		)
+	)
+	(wire
+		(pts
 			(xy 20.32 83.82) (xy 20.32 93.98)
 		)
@@
 		)
 	)
+	(hierarchical_label "Codec_SDA"
+		(shape input)
+		(at 121.92 63.5 180)
+		(fields_autoplaced yes)
+		(effects
+			(font
+				(size 1.27 1.27)
+			)
+			(justify right)
+		)
+	)
 	(hierarchical_label "+3,3V"
 		(shape input)
@@
 		)
 	)
+	(hierarchical_label "Codec_SCL"
+		(shape input)
+		(at 120.65 86.36 180)
+		(fields_autoplaced yes)
+		(effects
+			(font
+				(size 1.27 1.27)
+			)
+			(justify right)
+		)
+	)
 	(hierarchical_label "LED_SCL"
 		(shape input)
@@
 			)
 		)
-		(property "Footprint" ""
+		(property "Footprint" "Library:Switch carré"
 			(at 78.74 80.01 0)
 			(effects
@@
 			)
 		)
-		(property "Footprint" ""
+		(property "Footprint" "Library:Switch carré"
 			(at 78.74 133.35 0)
 			(effects
@@
 		(fields_autoplaced yes)
 		(property "Reference" "C1"
-			(at 116.84 52.0638 0)
+			(at 121.92 49.5235 0)
 			(effects
 				(font
 					(size 1.27 1.27)
 				)
-				(justify left)
+				(justify right)
 			)
 		)
-		(property "Value" "C_Small"
-			(at 116.84 49.5238 0)
+		(property "Value" "100nF"
+			(at 121.92 52.0635 0)
 			(effects
 				(font
 					(size 1.27 1.27)
 				)
-				(justify left)
+				(justify right)
 			)
 		)
-		(property "Footprint" ""
+		(property "Footprint" "Capacitor_SMD:C_0805_2012Metric_Pad1.18x1.45mm_HandSolder"
 			(at 119.38 50.8 0)
 			(effects
@@
 			)
 		)
-		(property "Footprint" ""
+		(property "Footprint" "Library:Switch carré"
 			(at 67.31 80.01 0)
 			(effects
@@
 			)
 		)
-		(property "Footprint" ""
+		(property "Footprint" "Capacitor_SMD:C_0805_2012Metric_Pad1.18x1.45mm_HandSolder"
 			(at 138.43 36.83 0)
 			(effects
@@
 			)
 		)
-		(property "Footprint" ""
+		(property "Footprint" "Resistor_SMD:R_0805_2012Metric_Pad1.20x1.40mm_HandSolder"
 			(at 217.932 125.73 90)
 			(effects
@@
 			)
 		)
-		(property "Footprint" ""
+		(property "Footprint" "Resistor_SMD:R_0805_2012Metric_Pad1.20x1.40mm_HandSolder"
 			(at 200.152 125.73 90)
 			(effects
@@
 			)
 		)
-		(property "Footprint" ""
+		(property "Footprint" "Library:Switch carré"
 			(at 55.88 80.01 0)
 			(effects
@@
 			)
 		)
-		(property "Footprint" ""
+		(property "Footprint" "Connector_PinHeader_1.27mm:PinHeader_2x07_P1.27mm_Vertical"
 			(at 240.03 76.2 0)
 			(effects
@@
 			)
 		)
-		(property "Footprint" ""
+		(property "Footprint" "Capacitor_SMD:C_0805_2012Metric_Pad1.18x1.45mm_HandSolder"
 			(at 148.59 39.37 0)
 			(effects
@@
 			)
 		)
-		(property "Footprint" ""
+		(property "Footprint" "Library:Switch carré"
 			(at 44.45 80.01 0)
 			(effects
@@
 			)
 		)
-		(property "Footprint" ""
+		(property "Footprint" "Library:Switch carré"
 			(at 67.31 133.35 0)
 			(effects
@@
 			)
 		)
-		(property "Footprint" ""
+		(property "Footprint" "Capacitor_SMD:C_0805_2012Metric_Pad1.18x1.45mm_HandSolder"
 			(at 151.13 36.83 0)
 			(effects
@@
 			)
 		)
-		(property "Footprint" ""
+		(property "Footprint" "Capacitor_SMD:C_0805_2012Metric_Pad1.18x1.45mm_HandSolder"
 			(at 146.05 41.91 0)
 			(effects
@@
 			)
 		)
-		(property "Footprint" ""
+		(property "Footprint" "Library:Switch carré"
 			(at 21.59 80.01 0)
 			(effects
@@
 			)
 		)
-		(property "Footprint" ""
+		(property "Footprint" "Library:Switch carré"
 			(at 33.02 80.01 0)
 			(effects
@@
 			)
 		)
-		(property "Footprint" ""
+		(property "Footprint" "Connector_Card:microSD_HC_Molex_104031-0811"
 			(at 292.1 130.81 0)
 			(effects
@@
 			)
 		)
-		(property "Footprint" ""
+		(property "Footprint" "Resistor_SMD:R_0805_2012Metric_Pad1.20x1.40mm_HandSolder"
 			(at 209.042 125.73 90)
 			(effects
@@
 			)
 		)
-		(property "Footprint" ""
+		(property "Footprint" "Capacitor_SMD:C_0805_2012Metric_Pad1.18x1.45mm_HandSolder"
 			(at 153.67 34.29 0)
 			(effects

Commit message: commit
Parts:
- C1, C12, C13, C14, C15, C2: footprint Capacitor_SMD:C_0805_2012Metric_Pad1.18x1.45mm_HandSolder -> Capacitor_SMD:C_0603_1608Metric_Pad1.08x0.95mm_HandSolder
Changed lines of the file:
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@@
 			)
 		)
-		(property "Footprint" "Capacitor_SMD:C_0805_2012Metric_Pad1.18x1.45mm_HandSolder"
+		(property "Footprint" "Capacitor_SMD:C_0603_1608Metric_Pad1.08x0.95mm_HandSolder"
 			(at 119.38 50.8 0)
 			(effects
@@
 			)
 		)
-		(property "Footprint" "Capacitor_SMD:C_0805_2012Metric_Pad1.18x1.45mm_HandSolder"
+		(property "Footprint" "Capacitor_SMD:C_0603_1608Metric_Pad1.08x0.95mm_HandSolder"
 			(at 138.43 36.83 0)
 			(effects
@@
 			)
 		)
-		(property "Footprint" "Capacitor_SMD:C_0805_2012Metric_Pad1.18x1.45mm_HandSolder"
+		(property "Footprint" "Capacitor_SMD:C_0603_1608Metric_Pad1.08x0.95mm_HandSolder"
 			(at 148.59 39.37 0)
 			(effects
@@
 			)
 		)
-		(property "Footprint" "Capacitor_SMD:C_0805_2012Metric_Pad1.18x1.45mm_HandSolder"
+		(property "Footprint" "Capacitor_SMD:C_0603_1608Metric_Pad1.08x0.95mm_HandSolder"
 			(at 151.13 36.83 0)
 			(effects
@@
 			)
 		)
-		(property "Footprint" "Capacitor_SMD:C_0805_2012Metric_Pad1.18x1.45mm_HandSolder"
+		(property "Footprint" "Capacitor_SMD:C_0603_1608Metric_Pad1.08x0.95mm_HandSolder"
 			(at 146.05 41.91 0)
 			(effects
@@
 			)
 		)
-		(property "Footprint" "Capacitor_SMD:C_0805_2012Metric_Pad1.18x1.45mm_HandSolder"
+		(property "Footprint" "Capacitor_SMD:C_0603_1608Metric_Pad1.08x0.95mm_HandSolder"
 			(at 153.67 34.29 0)
 			(effects
