File: hardware/gameflopMB_1/gameflopMB_1.kicad_pcb (KiCad board)
At the start: 2 copper layers, 182 x 94.5 mm, 76 parts, among them IC2 HTK16K33, IC6 HTK16K33, IC7 HTK16K33, IC8 HTK16K33, J1 AudioJack3, J2 USB_B_Micro, J3 Micro_SD_Card, J5 Conn_02x07_Odd_Even, J6 Conn_01x02, U1 TPS613222ADBV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

Commit message: commit
Parts:
- C1, C10, C11, C12, C13, C14, C15, C2, C3, C4, C5, C6, C7, C8, C9, C_Small1, C_Small10, C_Small2, C_Small3, C_Small4, C_Small5, C_Small6: footprint Capacitor_SMD:C_0805_2012Metric_Pad1.18x1.45mm_HandSolder -> Capacitor_SMD:C_0603_1608Metric_Pad1.08x0.95mm_HandSolder
- IC2, IC6, IC7: moved to B.Cu
- moved U16 151.6 mm to (80.7, 97.9)
- moved U17 151.6 mm to (80.7, 111.4)
- moved U18 151.6 mm to (94.2, 97.9)
- moved U19 151.6 mm to (94.2, 111.4)
- moved IC8 96.4 mm to (210.0, 86.0)
- moved IC7 80.1 mm to (193.4, 123.0), turned to 0 degrees
- moved IC6 63.3 mm to (146.8, 88.4), turned to 0 degrees
- moved IC2 62.5 mm to (147.3, 123.7), turned to 0 degrees
- moved D2 51.2 mm to (155.6, 149.6), turned to -90 degrees
- moved D3 49.6 mm to (157.5, 149.6), turned to -90 degrees
- moved C_Small10 46.7 mm to (146.8, 159.1)
- moved R13 43.3 mm to (143.8, 147.9)
- moved D1 43.1 mm to (163.6, 150.4), turned to 90 degrees
- moved U12 38.9 mm to (243.6, 87.0)
- moved U13 38.9 mm to (243.6, 100.5)
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Connections:
- IC2 pad 22: /Driver0/SCL -> Net-(IC2-ROW0/A2)
- IC2 pad 25: Net-(IC2-ROW13/K11) -> Net-(IC2-COM4)
- IC2 pad 26: Net-(IC2-ROW15/K13) -> Net-(IC2-COM5)
- IC2 pad 27: Net-(IC2-ROW14/K12) -> Net-(IC2-COM6)
- IC2 pad 6: Net-(IC2-COM4) -> Net-(IC2-COM7)
- IC2 pad 7: Net-(IC2-COM5) -> Net-(IC2-ROW15/K13)
- IC2 pad 8: Net-(IC2-COM6) -> Net-(IC2-ROW14/K12)
- IC2 pad 9: Net-(IC2-COM7) -> Net-(IC2-ROW13/K11)
- IC6 pad 22: /Driver0/SCL -> Net-(IC6-ROW0/A2)
- IC6 pad 25: Net-(IC6-ROW13/K11) -> Net-(IC6-COM4)
- IC6 pad 26: Net-(IC6-ROW15/K13) -> Net-(IC6-COM5)
- IC6 pad 27: Net-(IC6-ROW14/K12) -> Net-(IC6-COM6)
- IC6 pad 6: Net-(IC6-COM4) -> Net-(IC6-COM7)
- IC6 pad 7: Net-(IC6-COM5) -> Net-(IC6-ROW15/K13)
- IC6 pad 8: Net-(IC6-COM6) -> Net-(IC6-ROW14/K12)
- IC6 pad 9: Net-(IC6-COM7) -> Net-(IC6-ROW13/K11)
- IC8 pad 22: /Driver0/SCL -> Net-(IC8-ROW0/A2)
- U3 pad 12: Net-(IC2-COM1/KS0) -> Net-(IC2-COM0/AD)
- U3 pad 24: /Driver0/SCL -> Net-(IC2-ROW0/A2)
- U4 pad 11: Net-(IC6-ROW9/K7) -> Net-(IC6-ROW8/K6)
- U4 pad 24: /Driver0/SCL -> Net-(IC6-ROW0/A2)
- U7 pad 4: /Driver0/SCL -> Net-(IC7-ROW13/K11)
- U8 pad 24: /Driver0/SCL -> Net-(IC8-ROW0/A2)
Routing:
- net /Alim/+5V: track 0.00 -> 112.8 mm
- net +3.3V: track 213.1 -> 127.2 mm, vias 0 -> 6
- net Net-(IC2-ROW8/K6): track 0.00 -> 69.0 mm
- net Net-(J6-Pin_2): track 14.0 -> 78.4 mm
- net SPI1_SCK: track 0.00 -> 57.0 mm
- net Net-(IC8-COM7): track 0.00 -> 56.0 mm
- net /Driver0/SCL: track 0.00 -> 55.3 mm
- net Net-(IC8-COM0/AD): track 0.00 -> 55.3 mm
- net SPI1_MISO: track 0.00 -> 54.2 mm
- net Net-(IC8-ROW1/A1): track 0.00 -> 53.0 mm
- net Net-(IC8-COM6): track 0.00 -> 50.5 mm
- net A: track 0.00 -> 50.1 mm
- net Net-(IC6-ROW8/K6): track 0.00 -> 47.0 mm
- net Net-(IC8-ROW0/A2): track 0.00 -> 47.0 mm
- net Net-(IC8-COM1/KS0): track 0.00 -> 46.2 mm
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- added copper zone on In1.Cu, net +3.3V
- added copper zone on B.Cu, net GND
- added copper zone on F.Cu, net GND
- added copper zone on In2.Cu, net GND
Other:
- copper layers 2 -> 4

Commit message: last push hardware
Parts:
- moved U17 18.4 mm to (98.3, 116.5)
- moved U19 17.1 mm to (109.8, 104.5)
- moved U16 8.69 mm to (85.8, 104.9)
- moved U18 6.41 mm to (97.6, 92.5)
- moved J2 1.53 mm to (127.3, 159.5)
- moved J5 1.05 mm to (191.5, 160.7)
- moved J3 1.01 mm to (246.4, 138.5)
- moved J6 0.35 mm to (164.5, 160.2)
Routing:
- net /Driver0/SCL: track 55.3 -> 353.4 mm
- net /Alim/+5V: track 112.8 -> 399.8 mm, vias 0 -> 4
- net /Driver0/SDA: track 41.0 -> 321.9 mm, vias 0 -> 6
- net SelectO: track 0.00 -> 200.2 mm, vias 0 -> 2
- net Net-(C9-Pad2): track 0.00 -> 179.7 mm, vias 0 -> 2
- net Net-(C10-Pad2): track 0.00 -> 175.4 mm, vias 0 -> 4
- net Down: track 0.00 -> 170.8 mm, vias 0 -> 2
- net StartO: track 0.00 -> 170.2 mm, vias 0 -> 2
- net Right: track 0.00 -> 155.0 mm, vias 0 -> 2
- net SWDIO: track 0.00 -> 67.4 mm, vias 0 -> 2
- net SWDCK: track 0.00 -> 64.7 mm, vias 0 -> 2
- net +1V8: track 0.00 -> 56.1 mm, vias 0 -> 2
- net +3.3V: track 127.2 -> 79.3 mm, vias 6 -> 11
- net /Audio/I2C_SCL: track 0.00 -> 42.5 mm
- net /Audio/I2C_SDA: track 0.00 -> 42.2 mm, vias 0 -> 3
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